File: feikController pedal/feikController pedal.kicad_pcb (KiCad board)
At the start: 2 copper layers, 15.5 x 12.6 mm, 18 parts, among them U1 PIC16F18325-ISL

Commit message: updated schematic/PCB/gerber + added pics
Other:
- rule pad_to_mask_clearance: 0.05 -> 0
