File: feikController pedal/feikController pedal.sch (KiCad schematic (older format))
At the start: 18 parts, among them U1 PIC16F18325-ISL

Commit message: updated schematic/PCB/gerber + added pics
Parts:
- C1, C2, C3: symbol Device:CP1_Small -> Device:C_Polarized_Small_US
Changed lines of the file:
@@
 $EndComp
 $Comp
-L Device:CP1_Small C1
+L Device:C_Polarized_Small_US C1
 U 1 1 5DA2B48A
 P 5200 2150
@@
 	5200 2050 5200 2000
 $Comp
-L Device:CP1_Small C2
+L Device:C_Polarized_Small_US C2
 U 1 1 5DA61B3C
 P 5650 2150
@@
 VDD
 $Comp
-L Device:CP1_Small C3
+L Device:C_Polarized_Small_US C3
 U 1 1 5DABA497
 P 6050 2150
